Commit message: modified meshes paths in urdf

File: test_legs_urdf.urdf (robot description, URDF)
Before this commit: robot test_legs_urdf, 13 links, 12 joints
Links:
- link LAnkle: geometry collision mesh filename=package://meshes/LAnkle.STL; visual mesh filename=package://meshes/LAnkle.STL
- link LFemur: geometry collision mesh filename=package://meshes/LFemur.STL; visual mesh filename=package://meshes/LFemur.STL
- link LFoot: geometry collision mesh filename=package://meshes/LFoot.STL; visual mesh filename=package://meshes/LFoot.STL
- link LHip: geometry collision mesh filename=package://meshes/LHip.STL; visual mesh filename=package://meshes/LHip.STL
- link LLeg: geometry collision mesh filename=package://meshes/LLeg.STL; visual mesh filename=package://meshes/LLeg.STL
- link LTibia: geometry collision mesh filename=package://meshes/LTibia.STL; visual mesh filename=package://meshes/LTibia.STL
- link RAnkle: geometry collision mesh filename=package://meshes/RAnkle.STL; visual mesh filename=package://meshes/RAnkle.STL
- link RFemur: geometry collision mesh filename=package://meshes/RFemur.STL; visual mesh filename=package://meshes/RFemur.STL
- link RFoot: geometry collision mesh filename=package://meshes/RFoot.STL; visual mesh filename=package://meshes/RFoot.STL
- link RHip: geometry collision mesh filename=package://meshes/RHip.STL; visual mesh filename=package://meshes/RHip.STL
- link RLeg: geometry collision mesh filename=package://meshes/RLeg.STL; visual mesh filename=package://meshes/RLeg.STL
- link RTibia: geometry collision mesh filename=package://meshes/RTibia.STL; visual mesh filename=package://meshes/RTibia.STL
- link base_link: geometry collision mesh filename=package://meshes/base_link.STL; visual mesh filename=package://meshes/base_link.STL
