Commit message: updated link masses

File: NUBI_V4/NUBI_V4.urdf (robot description, URDF)
Before this commit: robot NUBI_V4, 20 links, 19 joints
Links:
- link L_A_1: mass 0.00270980906824082 -> 0.099
- link L_A_2: mass 0.0107696045304613 -> 0.026
- link L_N_1: mass 0.00406217499121926 -> 0.07
- link L_W_1: mass 0.117514351814221 -> 0.008
- link L_W_2: mass 0.000548582459427128 -> 0.099
- link L_W_3: mass 0.00416880860873112 -> 0.02
- link R_A_1: mass 0.00272881293242526 -> 0.099
- link R_A_2: mass 0.0107696045304606 -> 0.026
- link R_N_1: mass 0.00406217575218774 -> 0.07
- link R_W_1: mass 0.117514351814221 -> 0.008
- link R_W_2: mass 0.000534743192016889 -> 0.099
- link R_W_3: mass 0.00409019778386988 -> 0.02
- link Upper_body: mass 0.0205774766400463 -> 0.172
- link base_link: mass 0.00436456608198951 -> 0.108
- link hL_sh1: mass 0.00373121734305089 -> 0.005
- link hr_sh1: mass 0.00373121730714498 -> 0.005
