Commit message: Updated link masses with true masses

File: NUBI_V6/NUBI_V6.urdf (robot description, URDF)
Before this commit: robot NUBI_V6, 20 links, 19 joints
Links:
- link LAnkle: mass 1.70246844377126E-07 -> 0.099
- link LFemur: mass 0.00409019781377434 -> 0.02
- link LFoot: mass 0.0107696045359165 -> 0.026
- link LForearm: mass 8.51234221885626E-08 -> 0.0495
- link LHip: mass 1.70246844377133E-07 -> 0.099
- link LHumerus: mass 0.00754332256882732 -> 0.0545
- link LPelvis: mass 0.0862681975072362 -> 0.008
- link LShoulder: mass 0.00373121799749922 -> 0.005
- link LTibia: mass 0.00392507523860521 -> 0.07
- link RAnkle: mass 1.70246844377129E-07 -> 0.099
- link RFemur: mass 0.00409019740627706 -> 0.02
- link RFoot: mass 0.0107696045379167 -> 0.026
- link RForearm: mass 8.51234221885612E-08 -> 0.0495
- link RHip: mass 1.70246844377124E-07 -> 0.099
- link RHumerus: mass 0.00754330562120907 -> 0.0545
- link RPelvis: mass 0.086268 -> 0.008
- link RShoulder: mass 0.00373121795815298 -> 0.005
- link RTibia: mass 0.00392507494301407 -> 0.07
- link base_link: mass 0.0040904 -> 0.108
- link chest: mass 0.019754850289291 -> 0.172

Commit message: modified knee joint limits

File: NUBI_V6/NUBI_V6.urdf (robot description, URDF)
Before this commit: robot NUBI_V6, 20 links, 19 joints
Joints:
- joint LKnee_pitch: limit lower=-2.79 upper=2.79 effort=1.2 velocity=6.3 -> lower=-0.0175 upper=2.0071 effort=1.2 velocity=6.3
- joint RKnee_pitch: limit lower=-2.79 upper=2.79 effort=1.2 velocity=6.3 -> lower=-2.0071 upper=0.0175 effort=1.2 velocity=6.3

Commit message: fixed urdf axes to match physical robot

File: NUBI_V6/NUBI_V6.urdf (robot description, URDF)
Before this commit: robot NUBI_V6, 20 links, 19 joints
Joints:
- joint LAnkle_pitch: axis 0 -1 0 -> 0 1 0
- joint LAnkle_roll: axis 1 0 0 -> -1 0 0
- joint LHip_pitch: axis 1 0 0 -> -1 0 0
- joint RAnkle_pitch: axis 0 -1 0 -> 0 1 0
- joint RAnkle_roll: axis 0 -1 0 -> 0 1 0
