Commit message: organizational commit

File: view_robot_pkg/urdf/robot_description.urdf (robot description, URDF)
Before this commit: robot view_robot_pkg, 35 links, 34 joints
Links:
- removed link Right_finger_RG_joint
- removed link Right_gear_RG_joint
- removed link left_finger_LG_joint
- removed link left_finger_RG_joint
- removed link left_gear_LG_joint
- removed link left_gear_RG_joint
- removed link left_link_LG_joint
- removed link left_link_RG_joint
- removed link right_finger_LG_joint
- removed link right_gear_LG_joint
- removed link right_link_LG_joint
- removed link right_link_RG_joint
- added link left_finger_1, mass 0.00338679290688088; collision mesh filename=package://view_robot_pkg/meshes/left_finger_1.STL; visual mesh filename=package://view_robot_pkg/meshes/left_finger_1.STL
- added link left_finger_2, mass 0.00338679922396475; collision mesh filename=package://view_robot_pkg/meshes/left_finger_2.STL; visual mesh filename=package://view_robot_pkg/meshes/left_finger_2.STL
- added link left_finger_3, mass 0.0035965823618601; collision mesh filename=package://view_robot_pkg/meshes/left_finger_3.STL; visual mesh filename=package://view_robot_pkg/meshes/left_finger_3.STL
- added link right_finger_1, mass 0.00338658273554947; collision mesh filename=package://view_robot_pkg/meshes/right_finger_1.STL; visual mesh filename=package://view_robot_pkg/meshes/right_finger_1.STL
- added link right_finger_2, mass 0.00338655715396473; collision mesh filename=package://view_robot_pkg/meshes/right_finger_2.STL; visual mesh filename=package://view_robot_pkg/meshes/right_finger_2.STL
- added link right_finger_3, mass 0.00359633615394456; collision mesh filename=package://view_robot_pkg/meshes/right_finger_3.STL; visual mesh filename=package://view_robot_pkg/meshes/right_finger_3.STL
- link L_A_1: mass 0.00270980906824081 -> 0.0027098089897503
- link L_A_2: mass 0.0107696045304608 -> 0.010769604530461
- link L_N_1: mass 0.00406217499121926 -> 0.00406217499121864
- link L_W_1: mass 0.152073564561278 -> 0.158345120003422
- link L_W_2: mass 0.000548582459427165 -> 0.000548582459427157
- link L_W_3: mass 0.00416880860873003 -> 0.00416880860873036
- link R_A_1: mass 0.00272881286947315 -> 0.00272881293156423
- link R_A_2: mass 0.0107696045303586 -> 0.010769604530461
- link R_N_1: mass 0.00406217575232337 -> 0.00406217575228148
- link R_W_1: mass 0.152073564561278 -> 0.158345120003422
- link R_W_2: mass 0.00053474319201658 -> 0.000534743192016655
- link R_W_3: mass 0.00409019778385964 -> 0.00409019778392477
- link base_lin: mass 0.00436456608198958 -> 0.00436456608198957
- link hL_e: mass 0.0159991858724107 -> 0.0228146295779902
- link hL_sh1: mass 0.00373121734305147 -> 0.00373121734305094
- link hL_sh2: mass 0.0072690936477349 -> 0.00726909290807301
- link hr_e: mass 0.015999176996954 -> 0.0228149408605893
- link hr_sh1: mass 0.00373121730714512 -> 0.00373121732631075
- link hr_sh2: mass 0.00726909364773545 -> 0.00726909421290748
Joints:
- removed joint Right_finger_RG
- removed joint Right_gear_RG
- removed joint left_finger_LG
- removed joint left_finger_RG
- removed joint left_gear_LG
- removed joint left_gear_RG
- removed joint left_link_LG
- removed joint left_link_RG
- removed joint right_finger_LG
- removed joint right_gear_LG
- removed joint right_link_LG
- removed joint right_link_RG
- added joint left_finger_1_j: type revolute, parent hr_e, child left_finger_1, origin xyz=0.014539167438465 -0.0024548476567654 -0.0618153968254915 rpy=0.0377905175630072 -0.000102993744146965 0.0871190025831379, axis -0.996194698091742 0.0871557427477022 0, limit lower=-0.785 upper=0.785 effort=0 velocity=0
- added joint left_finger_2_j: type revolute, parent hr_e, child left_finger_2, origin xyz=-0.0186394892583865 -0.0053526740783667 -0.061818827028493 rpy=0.0377905175630072 -0.000102993744146965 0.0871190025831379, axis -0.996194698091746 -0.0871557427476552 0, limit lower=-0.785 upper=0.785 effort=0 velocity=0, mimic joint=left_finger_1_j multiplier=1 offset=0
- added joint left_finger_3_j: type revolute, parent hr_e, child left_finger_3, origin xyz=0.00440007245049012 -0.034655228822984 -0.0629962029174997 rpy=0.0377905175630072 -0.000102993744146965 0.0871190025831379, axis -1 0 0, limit lower=-0.785 upper=0.785 effort=0 velocity=0, mimic joint=left_finger_1_j multiplier=-1 offset=0
- added joint riggt_finger_1_j: type revolute, parent hL_e, child right_finger_1, origin xyz=-0.0345370835079564 -0.0630386544270789 0.0142975543144077 rpy=1.49108762194966 -1.48302409058719 -3.02562142764069, axis -0.996194698091741 -0.0871557427477142 0, limit lower=-0.785 upper=0.785 effort=0 velocity=0
- added joint right_finger_2_j: type revolute, parent hL_e, child right_finger_2, origin xyz=-0.031637194929915 -0.0627008349525799 -0.0188792025219854 rpy=1.49108762194966 -1.48302409058719 -3.02562142764069, axis -0.996194698091739 0.0871557427477304 0, limit lower=-0.785 upper=0.785 effort=0 velocity=0, mimic joint=riggt_finger_1_j multiplier=1 offset=0
- added joint right_finger_3_j: type revolute, parent hL_e, child right_finger_3, origin xyz=-0.00233480635832373 -0.0617898348928716 0.00417263981595195 rpy=1.49108762194966 -1.48302409058719 -3.02562142764069, axis -1 0 0, limit lower=-0.785 upper=0.785 effort=0 velocity=0, mimic joint=riggt_finger_1_j multiplier=-1 offset=0
- joint LAnkle_pitch: axis 0.00321902611343638 -0.999556505100927 -0.0296045770329757 -> 0.00321902611346478 -0.999556505100925 -0.0296045770330436; origin xyz=0.0116386736214952 0.00109273068918236 -0.0774847266386327 rpy=0 0 0 -> xyz=0.0116386736214943 0.00109273068918325 -0.0774847266386329 rpy=0 0 0
- joint LAnkle_roll: axis 0.999964392032425 0.00344846027439361 -0.00770212885881819 -> 0.99997044950115 0.00342421615064848 -0.00688294037617749; origin xyz=-0.0466491161038564 0.0211292222358059 0.000725339778560485 rpy=0 0 0 -> xyz=-0.0466491799896894 0.021130360108895 0.000687185849517435 rpy=0 0 0
- joint LHip_pitch: axis -0.0125726074067991 -0.999485937943567 -0.0294921921203482 -> -0.0125726074068017 -0.999485937943566 -0.029492192120357; origin xyz=0.0462337025626653 -0.0223530513381598 -0.00111240331126483 rpy=0 0 0 -> xyz=0.0462337025626542 -0.0223530513381598 -0.0011124033112655 rpy=0 0 0
- joint LHip_roll: axis 0.999896590427051 -0.0123609060710088 -0.00734958865932969 -> 0.999896590427052 -0.0123609060710002 -0.00734958865927157; origin xyz=-0.0350660356311487 0.00115022718562807 -0.0240322725212692 rpy=0 0 0 -> xyz=-0.0350660356311479 0.00115022718562807 -0.0240322725212685 rpy=0 0 0
- joint LHip_yaw: origin xyz=0.00811191095429442 0.0343859376847431 -0.0358999999999563 rpy=-0.0295865830615605 -0.00698131700551125 -0.231656625322495 -> xyz=0.00811191095683594 0.0343859376841071 -0.0358999999999909 rpy=-0.029586583062536 -0.00698131700797945 -0.231656625394124
- joint LKnee_pitch: axis 0.012572607406823 0.999485937943566 0.0294921921203551 -> 0.0125726074068399 0.999485937943568 0.0294921921202849
- joint Lelbow_roll: axis 0.999975614545494 2.6820905506732E-05 -0.00698352310799514 -> 0.000183244787815072 0.999529562327929 0.0306695362515648; origin xyz=-0.002073890762049 0.00190794827611906 -0.0678386008964182 rpy=0 0 0 -> xyz=-0.020812703098818 0.0210746679877154 -0.0671974588360775 rpy=0 0 0
- joint Lshoulder_pitch: axis -0.00018192577337194 -0.999562370008584 -0.0295809967011877 -> -0.000181925773373656 -0.999562370008605 -0.0295809967004767; origin xyz=0.00104096446219726 0.060169267832598 0.0298122840963835 rpy=0 0 0 -> xyz=0.00104096368704842 0.0601692528237647 0.0298122839682016 rpy=0 0 0
- joint Lshoulder_roll: axis 0.999975614156498 2.46709159308775E-05 -0.00698358673469515 -> 0.999994907013672 -8.75897164786316E-05 -0.00319034085315742; origin xyz=0.0190034845977193 0.0215910216665414 0.000506261459308988 rpy=0 0 0 -> xyz=0.0190038328299961 0.0215888829868018 0.000578333052573043 rpy=0 0 0
- joint RAnkle_pitch: axis -0.00321902611345547 0.999556505100927 0.0296045770329677 -> -0.00321902611345472 0.999556505100925 0.0296045770330376; origin xyz=0.0116621204095037 -0.000762059454564312 -0.0775407363717699 rpy=0 0 0 -> xyz=0.0116621204094988 -0.000762059454563868 -0.0775407363717717 rpy=0 0 0
- joint RAnkle_roll: axis 0.99997044950115 0.00342421615067466 -0.00688294037609805 -> 0.999970449501151 0.00342421615065541 -0.00688294037605934; origin xyz=-0.0464504790035918 -0.0206894543645093 -0.000414864266030435 rpy=0 0 0 -> xyz=-0.0464504790035913 -0.0206894543645093 -0.000414864266030657 rpy=0 0 0
- joint RHip_pitch: axis -0.0195011681197361 0.999368229569572 0.0297127273898547 -> -0.0195011681197689 0.999368229569573 0.0297127273898119; origin xyz=0.0461667822915901 0.0215038971400305 4.99520127628106E-05 rpy=0 0 0 -> xyz=0.0461667822915812 0.0215038971400434 4.99520127608122E-05 rpy=0 0 0
- joint RHip_roll: axis 0.999785460209647 0.019699590675994 -0.00639997504543661 -> 0.999785460209647 0.0196995906759968 -0.00639997504543753; origin xyz=-0.0344340076210223 0.00570690748207037 -0.0242946563290467 rpy=-0.0365680701988691 -0.00698114687545119 -0.188554812891601 -> xyz=-0.0344340076210214 0.00570690748207126 -0.0242946563290465 rpy=-0.0365680701988691 -0.00698114687545119 -0.188554812891601
- joint RHip_yaw: axis -0.00130889829658463 -0.00685746167291572 -0.999975630705396 -> -0.0013088982966226 -0.00685746167288035 -0.999975630705396; origin xyz=-0.00811115881539393 -0.034382750486029 -0.0359000000000256 rpy=0.00685752129495438 -0.00130889866810499 -0.0430575611663204 -> xyz=-0.00811115881777424 -0.0343827504855072 -0.0358999999999901 rpy=0.00685752129353344 -0.00130889867034655 -0.0430575612379543
- joint RKnee_pitch: axis 0.0195011681198009 -0.999368229569575 -0.0297127273897283 -> 0.019501168119795 -0.999368229569574 -0.0297127273897501; origin xyz=-0.0122292736907317 0.00158734307245378 -0.0774034293266377 rpy=0 0 0 -> xyz=-0.0122292736907312 0.00158734307245423 -0.0774034293266375 rpy=0 0 0
- joint Relbow_roll: axis 2.6821E-05 -0.0069835 0.99998 -> 0.999562369953202 0.0295810117224753 0.000179774894971738; origin xyz=0.0019079 -0.067834 -0.0027738 rpy=0 0 0 -> xyz=0.0209990879193984 -0.0671360220957142 -0.0217699501600307 rpy=0 0 0
- joint Rshoulder_pitch: axis 0.000181925773391679 0.999562370008603 0.0295809967005423 -> 0.000181925773392807 0.999562370008612 0.0295809967002308; origin xyz=0.00101152037119112 -0.101559924097068 0.0250260965550666 rpy=0 0 0 -> xyz=0.00101152047504471 -0.101559945328362 0.0250260707046959 rpy=0 0 0
- joint Rshoulder_roll: origin xyz=0.01899560198786 -0.0215900909300901 -0.000771639290922721 rpy=1.5707963267949 0 1.5707963267949 -> xyz=0.0189956054092215 -0.0215900780747444 -0.000771635444381857 rpy=1.5707963267949 0 1.5707963267949
- joint Upper_body_joint: limit lower=0 upper=0 effort=1.2 velocity=0 -> lower=0.0 upper=0.0 effort=1.2 velocity=6.3; origin xyz=0.0155859734030666 0.0150977984615721 0.0154999999999887 rpy=-0.0295865830615605 -0.00698131700551125 -0.231656625322495 -> xyz=0.0155859734041142 0.0150977984604785 0.0155000000000001 rpy=-0.029586583062536 -0.00698131700797945 -0.231656625394124
- joint camera_joint: origin xyz=0.0 -0.019 0.04 rpy=0 0 0 -> xyz=0.00675 -0.0185 0.10635 rpy=0 0 0
- joint left_arm_tcp_joint: origin xyz=0 -0.0026 -0.1 rpy=0 0 0 -> xyz=0.00007 -0.01679 -0.0733 rpy=0 0 0
- joint right_arm_tcp_joint: origin xyz=0.006 -0.1 0 rpy=0 0 0 -> xyz=-0.01957 -0.07339 -0.00155 rpy=0 0 0
